File: corne-ultralight/pcb/corne-ultralight.kicad_pcb (KiCad board)
At the start: 2 copper layers, 275.5 x 105.6 mm, 132 parts, among them J2 OLED, J5 Breakaway_Tabs, J7 OLED, SW1 SW_PUSH, SW10 SW_PUSH, SW11 SW_PUSH, SW12 SW_PUSH, SW13 SW_PUSH, SW14 SW_PUSH, SW15 SW_PUSH, SW16 SW_PUSH, SW17 SW_PUSH, SW18 SW_PUSH, SW19 SW_PUSH, SW2 SW_PUSH, SW20 SW_PUSH, SW21 SW_PUSH, SW22 SW_PUSH, SW23 SW_PUSH, SW24 SW_PUSH, SW25 SW_PUSH, SW26 SW_PUSH, SW27 SW_PUSH, SW28 SW_PUSH, SW29 SW_PUSH, SW3 SW_PUSH, SW30 SW_PUSH, SW31 SW_PUSH, SW32 SW_PUSH, SW33 SW_PUSH, SW34 SW_PUSH, SW35 SW_PUSH, SW36 SW_PUSH, SW37 SW_PUSH, SW38 SW_PUSH, SW39 SW_PUSH, SW4 SW_PUSH, SW40 SW_PUSH, SW41 SW_PUSH, SW42 SW_PUSH, SW5 SW_PUSH, SW6 SW_PUSH, SW7 SW_PUSH, SW8 SW_PUSH, SW9 SW_PUSH, U1 ProMicro, U2 ProMicro

Commit message: Choc v1 hotswap
Parts:
- D1, D10, D11, D12, D13, D14, D15, D16, D17, D18, D19, D2, D20, D21, D22, D23, D24, D25, D26, D27, D28, D29, D3, D30, D31, D32, D33, D34, D35, D36, D37, D38, D39, D4, D40, D41, D42, D5, D6, D7, D8, D9: footprint kbd:D3_TH_SMD_v2 -> kbd:D3_TH
- SW1, SW10, SW11, SW12, SW13, SW14, SW15, SW16, SW17, SW18, SW19, SW2, SW20, SW22, SW23, SW24, SW25, SW26, SW27, SW28, SW29, SW3, SW30, SW31, SW32, SW33, SW34, SW35, SW36, SW37, SW38, SW39, SW4, SW40, SW41, SW5, SW6, SW7, SW8, SW9: footprint gateron-ks27:gateron-ks27-choc-v1-mx -> ScottoKeebs_Hotswap:Hotswap_Choc_V1_Flipped
- SW21, SW42: footprint gateron-ks27:gateron-ks27-choc-v1-mx-1.5u -> ScottoKeebs_Hotswap:Hotswap_Choc_V1_1.50u
- moved D15 9.78 mm to (71.2, 88.2)
- moved D16 9.76 mm to (68.2, 88.2)
- moved D3 4.20 mm to (68.2, 36.7), turned to -90 degrees
- moved D4 4.20 mm to (71.2, 36.7), turned to -90 degrees
- moved D10 4.00 mm to (71.2, 55.9), turned to -90 degrees
- moved D9 4.00 mm to (68.2, 55.9)
- moved D2 3.00 mm to (33.3, 42.9), turned to -90 degrees
- moved D7 3.00 mm to (30.2, 61.9), turned to -90 degrees
- moved D13 3.00 mm to (30.2, 80.9), turned to -90 degrees
- moved D14 3.00 mm to (33.2, 80.9), turned to -90 degrees
- moved D19 3.00 mm to (80.5, 95.9), turned to -90 degrees
- moved D8 3.00 mm to (33.2, 61.9), turned to -90 degrees
- moved D1 2.97 mm to (30.2, 42.9), turned to -90 degrees
- moved D28 2.00 mm to (270.7, 62.9)
- moved D29 2.00 mm to (267.7, 62.9)
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Routing:
- net col3_r: track 149.9 -> 74.9 mm
- net col4_r: track 129.4 -> 55.1 mm
- net row2_r: track 139.2 -> 92.8 mm
- net row3_r: track 88.1 -> 45.7 mm
- net row0_r: track 131.2 -> 92.2 mm
- net col5_r: track 115.8 -> 91.2 mm
- net Net-(D21-A): track 42.4 -> 64.8 mm
- net col5: track 91.2 -> 112.3 mm, vias 1 -> 5
- net Net-(D40-A): track 21.5 -> 1.23 mm, vias 1 -> 0
- net Net-(D29-A): track 23.0 -> 40.9 mm, vias 1 -> 0
- net col0: track 177.7 -> 160.0 mm, vias 1 -> 4
- net Net-(D31-A): track 17.4 -> 0.00 mm
- net row3: track 97.9 -> 82.3 mm
- net Net-(D8-A): track 8.17 -> 22.7 mm, vias 0 -> 2
- net Net-(D37-A): track 14.2 -> 0.00 mm
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
Commit message: Switch to SMD only diodes, Finish routing
Parts:
- D1, D10, D11, D12, D13, D14, D15, D16, D17, D18, D19, D2, D20, D21, D22, D23, D24, D25, D26, D27, D28, D29, D3, D30, D31, D32, D33, D34, D35, D36, D37, D38, D39, D4, D40, D41, D42, D5, D6, D7, D8, D9: footprint kbd:D3_TH -> ScottoKeebs_Components:Diode_SOD-123
- moved D27 13.9 mm to (183.9, 50.4), turned to 0 degrees
- moved D33 9.44 mm to (183.9, 52.8), turned to 0 degrees
- turned D26 to -90 degrees
- turned D32 to -90 degrees
- turned D38 to -90 degrees
- turned D40 to -90 degrees
- turned D41 to -90 degrees
- turned D42 to -90 degrees
- turned SW27 to 180 degrees
- turned SW33 to 180 degrees
Routing:
- net col4_r: track 55.1 -> 154.5 mm, vias 1 -> 3
- net col3_r: track 74.9 -> 148.4 mm, vias 1 -> 2
- net row0_r: track 92.2 -> 159.1 mm
- net row2_r: track 92.8 -> 153.6 mm, vias 2 -> 4
- net row3_r: track 45.7 -> 73.8 mm
- net col5_r: track 91.2 -> 115.0 mm, vias 1 -> 4
- net Net-(D31-A): track 0.00 -> 22.2 mm, vias 0 -> 2
- net Net-(D37-A): track 0.00 -> 22.0 mm, vias 0 -> 2
- net Net-(D40-A): track 1.23 -> 20.4 mm
- net row1_r: track 128.8 -> 145.6 mm
- net Net-(D42-A): track 41.1 -> 31.5 mm
- net Net-(D33-A): track 18.2 -> 9.02 mm
- net Net-(D36-A): track 0.00 -> 8.90 mm
- net Net-(D41-A): track 19.1 -> 25.5 mm
- net Net-(D12-A): track 0.00 -> 4.86 mm
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Other:
- board text added: "Corne UltraLight v2.0 PCB Wireless Hotswap Choc V1 Designed by foostan, mods by petejohanson & ber2go"
- board text removed: "Corne Light v2.0 PCB Designed by foostan"
- board text removed: "Corne UltraLight v2.0 PCB Designed by foostan, mods by petejohanson"
